Commit message: fix controller vehicle params

File: rsc/ouzel/temp.urdf (robot description, URDF)
Before this commit: robot ouzel, 27 links, 26 joints
Links:
- removed link ouzel/force_sensor_tool
- removed link ouzel/manipulator
- removed link ouzel/tool
Joints:
- removed joint ouzel/force_sensor_tool
- removed joint ouzel/manipulator_joint
- removed joint ouzel/tool_joint
