Commit message: hook_ref_{left/right} sensors

File: rsc/ouzel/temp_hook.urdf (robot description, URDF)
Before this commit: robot ouzel, 29 links, 28 joints
Links:
- removed link hook_ref
- added link hook_ref_left, mass 0; visual sphere radius=0.015
- added link hook_ref_right, mass 0; visual sphere radius=0.015
Joints:
- removed joint hook_ref
- added joint hook_ref_left: type fixed, parent hook, child hook_ref_left, origin xyz=0 0 -0.0375 rpy=0 0 0
- added joint hook_ref_right: type fixed, parent hook, child hook_ref_right, origin xyz=0 0 0.0375 rpy=0 0 0
