Commit message: add ouzel_simple.obj

File: rsc/ouzel_delta/temp.urdf (robot description, URDF)
Before this commit: robot ouzel, 27 links, 26 joints
Links:
- link ouzel/tilt_unit_0: geometry collision box size=0.005 0.005 0.005; visual mesh filename=/home/vincent/rl_4_aerial_manipulator/catkin_ws/src/rotors_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 scale=1 1 1
- link ouzel/tilt_unit_1: geometry collision box size=0.005 0.005 0.005; visual mesh filename=/home/vincent/rl_4_aerial_manipulator/catkin_ws/src/rotors_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 scale=1 1 1
- link ouzel/tilt_unit_2: geometry collision box size=0.005 0.005 0.005; visual mesh filename=/home/vincent/rl_4_aerial_manipulator/catkin_ws/src/rotors_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 scale=1 1 1
- link ouzel/tilt_unit_3: geometry collision box size=0.005 0.005 0.005; visual mesh filename=/home/vincent/rl_4_aerial_manipulator/catkin_ws/src/rotors_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 scale=1 1 1
- link ouzel/tilt_unit_4: geometry collision box size=0.005 0.005 0.005; visual mesh filename=/home/vincent/rl_4_aerial_manipulator/catkin_ws/src/rotors_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 scale=1 1 1
- link ouzel/tilt_unit_5: geometry collision box size=0.005 0.005 0.005; visual mesh filename=/home/vincent/rl_4_aerial_manipulator/catkin_ws/src/rotors_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 scale=1 1 1
- link rotor_0: geometry collision cylinder length=0.005 radius=0.1143; visual mesh filename=/home/vincent/rl_4_aerial_manipulator/catkin_ws/src/rotors_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 scale=0.1143 0.1143 0.1143
- link rotor_1: geometry collision cylinder length=0.005 radius=0.1143; visual mesh filename=/home/vincent/rl_4_aerial_manipulator/catkin_ws/src/rotors_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 scale=0.1143 0.1143 0.1143
- link rotor_10: geometry collision cylinder length=0.005 radius=0.1143; visual mesh filename=/home/vincent/rl_4_aerial_manipulator/catkin_ws/src/rotors_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 scale=0.1143 0.1143 0.1143
- link rotor_11: geometry collision cylinder length=0.005 radius=0.1143; visual mesh filename=/home/vincent/rl_4_aerial_manipulator/catkin_ws/src/rotors_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 scale=0.1143 0.1143 0.1143
- link rotor_2: geometry collision cylinder length=0.005 radius=0.1143; visual mesh filename=/home/vincent/rl_4_aerial_manipulator/catkin_ws/src/rotors_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 scale=0.1143 0.1143 0.1143
- link rotor_3: geometry collision cylinder length=0.005 radius=0.1143; visual mesh filename=/home/vincent/rl_4_aerial_manipulator/catkin_ws/src/rotors_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 scale=0.1143 0.1143 0.1143
- link rotor_4: geometry collision cylinder length=0.005 radius=0.1143; visual mesh filename=/home/vincent/rl_4_aerial_manipulator/catkin_ws/src/rotors_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 scale=0.1143 0.1143 0.1143
- link rotor_5: geometry collision cylinder length=0.005 radius=0.1143; visual mesh filename=/home/vincent/rl_4_aerial_manipulator/catkin_ws/src/rotors_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 scale=0.1143 0.1143 0.1143
- link rotor_6: geometry collision cylinder length=0.005 radius=0.1143; visual mesh filename=/home/vincent/rl_4_aerial_manipulator/catkin_ws/src/rotors_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 scale=0.1143 0.1143 0.1143
- link rotor_7: geometry collision cylinder length=0.005 radius=0.1143; visual mesh filename=/home/vincent/rl_4_aerial_manipulator/catkin_ws/src/rotors_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 scale=0.1143 0.1143 0.1143
- link rotor_8: geometry collision cylinder length=0.005 radius=0.1143; visual mesh filename=/home/vincent/rl_4_aerial_manipulator/catkin_ws/src/rotors_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 scale=0.1143 0.1143 0.1143
- link rotor_9: geometry collision cylinder length=0.005 radius=0.1143; visual mesh filename=/home/vincent/rl_4_aerial_manipulator/catkin_ws/src/rotors_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 scale=0.1143 0.1143 0.1143

Commit message: fix delta arm

File: rsc/ouzel_delta/temp.urdf (robot description, URDF)
Before this commit: robot ouzel, 27 links, 26 joints
Links:
- removed link ouzel/force_sensor_tool
- removed link ouzel/manipulator
- removed link ouzel/tool
- added link delta/delta_base_link, mass 0.25
- added link delta/delta_link1_0, mass 0.041; collision box size=0.1558227 0.019 0.01; visual box size=0.1558227 0.019 0.01
- added link delta/delta_link1_1, mass 0.041; collision box size=0.1558227 0.019 0.01; visual box size=0.1558227 0.019 0.01
- added link delta/delta_link1_2, mass 0.041; collision box size=0.1558227 0.019 0.01; visual box size=0.1558227 0.019 0.01
Joints:
- removed joint ouzel/force_sensor_tool
- removed joint ouzel/manipulator_joint
- removed joint ouzel/tool_joint
- added joint delta/delta_joint_upper_0: type continuous, parent delta/delta_base_link, child delta/delta_link1_0, origin xyz=0.0743656 0.0 0.0 rpy=0.0 0.0 0, axis 0.0 1.0 0.0, limit lower=-1.570796326795 upper=1.570796326795 effort=10.0 velocity=5.0
- added joint delta/delta_joint_upper_1: type continuous, parent delta/delta_base_link, child delta/delta_link1_1, origin xyz=-0.037182800000008884 0.06440249876766692 0.0 rpy=0.0 0.0 2.0943951023933334, axis 0.0 1.0 0.0, limit lower=-1.570796326795 upper=1.570796326795 effort=10.0 velocity=5.0
- added joint delta/delta_joint_upper_2: type continuous, parent delta/delta_base_link, child delta/delta_link1_2, origin xyz=-0.037182799999982245 -0.06440249876768231 0.0 rpy=0.0 0.0 4.188790204786667, axis 0.0 1.0 0.0, limit lower=-1.570796326795 upper=1.570796326795 effort=10.0 velocity=5.0
- added joint mounting_joint: type fixed, parent ouzel/base_link, child delta/delta_base_link, origin xyz=0 0 0.073 rpy=0.0 0.0 0.0
- joint ouzel/tilt_unit_2_revolutejoint: origin xyz=0.259807621135 0.15 0 rpy=0 0 0.52359877559 -> xyz=0.25980762113519995 0.15 0 rpy=0 0 0.52359877559
- joint ouzel/tilt_unit_3_revolutejoint: origin xyz=-0.259807621135 -0.15 0 rpy=0 0 3.66519142919 -> xyz=-0.25980762113519995 -0.15 0 rpy=0 0 3.66519142919
- joint ouzel/tilt_unit_4_revolutejoint: origin xyz=0.259807621135 -0.15 0 rpy=0 0 5.75958653158 -> xyz=0.25980762113519995 -0.15 0 rpy=0 0 5.75958653158
- joint ouzel/tilt_unit_5_revolutejoint: origin xyz=-0.259807621135 0.15 0 rpy=0 0 2.61799387799 -> xyz=-0.25980762113519995 0.15 0 rpy=0 0 2.61799387799

Commit message: fix vehicle params

File: rsc/ouzel_delta/temp.urdf (robot description, URDF)
Before this commit: robot ouzel, 28 links, 27 joints
Links:
- removed link delta/delta_base_link
- removed link delta/delta_link1_0
- removed link delta/delta_link1_1
- removed link delta/delta_link1_2
Joints:
- removed joint delta/delta_joint_upper_0
- removed joint delta/delta_joint_upper_1
- removed joint delta/delta_joint_upper_2
- removed joint mounting_joint
