Commit message: handle ref to track posiion of the handle

File: rsc/objectInteraction/model.urdf (robot description, URDF)
Before this commit: robot shelf, 11 links, 10 joints
Links:
- link handle_ref: mass 0.01 -> 0.0
Joints:
- joint handle_ref: origin xyz=-0.0405 0 0 rpy=0 0 0 -> xyz=-0.050 0 0 rpy=0 0 0
